File: pcb/VLT.kicad_pcb (KiCad board)
At the start: 2 copper layers, 44.9 x 18.3 mm, 54 parts, among them J1 USB_C_Receptacle, Q2 AO3416A, SW1 SW_MEC_5E, SW2 SW_MEC_5E, SW3 SW_DIP_x02, U1 ATtiny1604-SS, U2 FT232RL, U3 AT24CM02-SSHM, U4 RNG90, U5 74AHCT1G00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

Commit message: Adapt values for rng
Parts:
- C12: value 1n -> 1u
- C13: value 10n -> 10u
- C7, C8, C9: value 100n -> n.B.
- R19, R20: value 10k -> 47k
Changed lines of the file:
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@@
     (property "Sheetfile" "VLT.kicad_sch")
     (property "Sheetname" "")
-    (property "Vendor" "HTL")
-    (property "VendorId" "100128")
+    (property "Vendor" "")
+    (property "VendorId" "")
     (property "ki_description" "Unpolarized capacitor")
     (property "ki_keywords" "cap capacitor")
@@
         (effects (font (size 0.6 0.6) (thickness 0.12)))
     )
-    (fp_text value "100n" (at 0 1.85) (layer "F.Fab")
+    (fp_text value "n.B." (at 0 1.85) (layer "F.Fab")
         (effects (font (size 1 1) (thickness 0.15)))
     )
@@
     (property "Sheetfile" "VLT.kicad_sch")
     (property "Sheetname" "")
-    (property "Vendor" "HTL")
-    (property "VendorId" "100128")
+    (property "Vendor" "")
+    (property "VendorId" "")
     (property "ki_description" "Unpolarized capacitor")
     (property "ki_keywords" "cap capacitor")
@@
         (effects (font (size 0.6 0.6) (thickness 0.12)))
     )
-    (fp_text value "100n" (at 0 -1.6764) (layer "F.Fab")
+    (fp_text value "n.B." (at 0 -1.6764) (layer "F.Fab")
         (effects (font (size 1 1) (thickness 0.15)))
     )
@@
     (property "Sheetfile" "VLT.kicad_sch")
     (property "Sheetname" "")
-    (property "Vendor" "HTL")
-    (property "VendorId" "100128")
+    (property "Vendor" "")
+    (property "VendorId" "")
     (property "ki_description" "Unpolarized capacitor")
     (property "ki_keywords" "cap capacitor")
@@
         (effects (font (size 0.6 0.6) (thickness 0.12)))
     )
-    (fp_text value "100n" (at 1.2936 2.8194 90) (layer "F.Fab")
+    (fp_text value "n.B." (at 1.2936 2.8194 90) (layer "F.Fab")
         (effects (font (size 1 1) (thickness 0.15)))
     )
@@
     (property "Sheetname" "")
     (property "Vendor" "HTL")
-    (property "VendorId" "102542")
+    (property "VendorId" "100134")
     (property "ki_description" "Unpolarized capacitor")
     (property "ki_keywords" "cap capacitor")
@@
         (effects (font (size 0.6 0.6) (thickness 0.12)) (justify mirror))
     )
-    (fp_text value "1n" (at 2.8466 0.0126 90) (layer "B.Fab")
+    (fp_text value "1u" (at 2.8466 0.0126 90) (layer "B.Fab")
         (effects (font (size 1 1) (thickness 0.15)) (justify mirror))
     )
@@
     (property "Sheetname" "")
     (property "Vendor" "HTL")
-    (property "VendorId" "102538")
+    (property "VendorId" "100138")
     (property "ki_description" "Unpolarized capacitor")
     (property "ki_keywords" "cap capacitor")
@@
         (effects (font (size 0.6 0.6) (thickness 0.12)) (justify mirror))
     )
-    (fp_text value "10n" (at -3.1224 0.0655) (layer "B.Fab")
+    (fp_text value "10u" (at -3.1224 0.0655) (layer "B.Fab")
         (effects (font (size 1 1) (thickness 0.15)) (justify mirror))
     )
@@
     (property "Sheetname" "")
     (property "Vendor" "HTL")
-    (property "VendorId" "102967")
+    (property "VendorId" "102980")
     (property "ki_description" "Resistor")
     (property "ki_keywords" "R res resistor")
@@
         (effects (font (size 0.6 0.6) (thickness 0.12)) (justify mirror))
     )
-    (fp_text value "10k" (at 1.143 1.6654 90) (layer "B.Fab")
+    (fp_text value "47k" (at 1.143 1.6654 90) (layer "B.Fab")
         (effects (font (size 1 1) (thickness 0.15)) (justify mirror))
     )
@@
     (property "Sheetname" "")
     (property "Vendor" "HTL")
-    (property "VendorId" "102967")
+    (property "VendorId" "102980")
     (property "ki_description" "Resistor")
     (property "ki_keywords" "R res resistor")
@@
         (effects (font (size 0.6 0.6) (thickness 0.12)) (justify mirror))
     )
-    (fp_text value "10k" (at -3.0615 -0.0144 90) (layer "B.Fab")
-        (effects (font (size 1 1) (thickness 0.15)) (justify mirror))
-    )
+    (fp_text value "47k" (at -3.0615 -0.0144 90) (layer "B.Fab")
+        (effects (font (size 1 1) (thickness 0.15)) (justify mirror))
+    )
