File: pcb/VLT.kicad_pcb (KiCad board)
At the start: 2 copper layers, 44.9 x 18.3 mm, 54 parts, among them J1 USB_C_Receptacle, Q2 AO3416A, SW1 SW_MEC_5E, SW2 SW_MEC_5E, SW3 SW_DIP_x02, U1 ATtiny1604-SS, U2 FT232RL, U3 AT24CM02-SSHM, U4 RNG90, U5 74AHCT1G00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

Commit message: Update to KiCAD 9
Other:
- outline, holes or cut-outs redrawn
