File: pcb/VLT.kicad_sch (KiCad schematic)
At the start: 54 parts, among them J1 USB_C_Receptacle, Q2 AO3416A, SW1 SW_MEC_5E, SW2 SW_MEC_5E, SW3 SW_DIP_x02, U1 ATtiny1604-SS, U2 FT232RL, U3 AT24CM02-SSHM, U4 RNG90, U5 74AHCT1G00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

Commit message: Change partlist vendors
Parts:
- C1, C2: Vendor DigiKey -> HTL; VendorId 478-1673-1-ND -> 103620
- SW1, SW2: Vendor DigiKey -> HTL; VendorId CKN10891CT-ND -> 103586
- SW3: Vendor DigiKey -> HTL; VendorId CT2192LPST-ND -> 103604
- U1: Vendor DigiKey -> HTL; VendorId ATTINY1604-SSNRCT-ND -> 103615
- U3: Vendor DigiKey -> HTL; VendorId AT24CM02-SSHM-TCT-ND -> 103616
- U4: Vendor DigiKey -> HTL; VendorId 150-RNG90-SSVDA-TCT-ND -> 103617
- U5, U6: Vendor DigiKey -> HTL; VendorId 296-1111-1-ND -> 103618
- U7: Vendor DigiKey -> HTL; VendorId 296-4714-1-ND -> 103619
Changed lines of the file:
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@@
       (effects (font (size 1.27 1.27)) hide)
     )
-    (property "Vendor" "DigiKey" (at 199.39 54.61 0)
-      (effects (font (size 1.27 1.27)) hide)
-    )
-    (property "VendorId" "ATTINY1604-SSNRCT-ND" (at 199.39 54.61 0)
+    (property "Vendor" "HTL" (at 199.39 54.61 0)
+      (effects (font (size 1.27 1.27)) hide)
+    )
+    (property "VendorId" "103615" (at 199.39 54.61 0)
       (effects (font (size 1.27 1.27)) hide)
     )
@@
       (effects (font (size 1.27 1.27)) hide)
     )
-    (property "Vendor" "DigiKey" (at 25.4 177.8 0)
-      (effects (font (size 1.27 1.27)) hide)
-    )
-    (property "VendorId" "478-1673-1-ND" (at 25.4 177.8 0)
+    (property "Vendor" "HTL" (at 25.4 177.8 0)
+      (effects (font (size 1.27 1.27)) hide)
+    )
+    (property "VendorId" "103620" (at 25.4 177.8 0)
       (effects (font (size 1.27 1.27)) hide)
     )
@@
       (effects (font (size 1.27 1.27)) hide)
     )
-    (property "Vendor" "DigiKey" (at 171.45 66.04 0)
-      (effects (font (size 1.27 1.27)) hide)
-    )
-    (property "VendorId" "CKN10891CT-ND" (at 171.45 66.04 0)
+    (property "Vendor" "HTL" (at 171.45 66.04 0)
+      (effects (font (size 1.27 1.27)) hide)
+    )
+    (property "VendorId" "103586" (at 171.45 66.04 0)
       (effects (font (size 1.27 1.27)) hide)
     )
@@
       (effects (font (size 1.27 1.27)) hide)
     )
-    (property "Vendor" "DigiKey" (at 256.54 46.99 0)
-      (effects (font (size 1.27 1.27)) hide)
-    )
-    (property "VendorId" "AT24CM02-SSHM-TCT-ND" (at 256.54 46.99 0)
+    (property "Vendor" "HTL" (at 256.54 46.99 0)
+      (effects (font (size 1.27 1.27)) hide)
+    )
+    (property "VendorId" "103616" (at 256.54 46.99 0)
       (effects (font (size 1.27 1.27)) hide)
     )
@@
       (effects (font (size 1.27 1.27)) hide)
     )
-    (property "Vendor" "DigiKey" (at 38.1 177.8 0)
-      (effects (font (size 1.27 1.27)) hide)
-    )
-    (property "VendorId" "478-1673-1-ND" (at 38.1 177.8 0)
+    (property "Vendor" "HTL" (at 38.1 177.8 0)
+      (effects (font (size 1.27 1.27)) hide)
+    )
+    (property "VendorId" "103620" (at 38.1 177.8 0)
       (effects (font (size 1.27 1.27)) hide)
     )
@@
       (effects (font (size 1.27 1.27)) hide)
     )
-    (property "Vendor" "DigiKey" (at 196.85 119.38 0)
-      (effects (font (size 1.27 1.27)) hide)
-    )
-    (property "VendorId" "296-1111-1-ND" (at 196.85 119.38 0)
+    (property "Vendor" "HTL" (at 196.85 119.38 0)
+      (effects (font (size 1.27 1.27)) hide)
+    )
+    (property "VendorId" "103618" (at 196.85 119.38 0)
       (effects (font (size 1.27 1.27)) hide)
     )
@@
       (effects (font (size 1.27 1.27)) hide)
     )
-    (property "Vendor" "DigiKey" (at 256.54 82.55 0)
-      (effects (font (size 1.27 1.27)) hide)
-    )
-    (property "VendorId" "150-RNG90-SSVDA-TCT-ND" (at 256.54 82.55 0)
+    (property "Vendor" "HTL" (at 256.54 82.55 0)
+      (effects (font (size 1.27 1.27)) hide)
+    )
+    (property "VendorId" "103617" (at 256.54 82.55 0)
       (effects (font (size 1.27 1.27)) hide)
     )
@@
       (effects (font (size 1.27 1.27)) hide)
     )
-    (property "Vendor" "DigiKey" (at 247.65 119.38 0)
-      (effects (font (size 1.27 1.27)) hide)
-    )
-    (property "VendorId" "296-1111-1-ND" (at 247.65 119.38 0)
+    (property "Vendor" "HTL" (at 247.65 119.38 0)
+      (effects (font (size 1.27 1.27)) hide)
+    )
+    (property "VendorId" "103618" (at 247.65 119.38 0)
       (effects (font (size 1.27 1.27)) hide)
     )
@@
       (effects (font (size 1.27 1.27)) hide)
     )
-    (property "Vendor" "DigiKey" (at 222.25 88.9 0)
-      (effects (font (size 1.27 1.27)) hide)
-    )
-    (property "VendorId" "296-4714-1-ND" (at 222.25 88.9 0)
+    (property "Vendor" "HTL" (at 222.25 88.9 0)
+      (effects (font (size 1.27 1.27)) hide)
+    )
+    (property "VendorId" "103619" (at 222.25 88.9 0)
       (effects (font (size 1.27 1.27)) hide)
     )
@@
       (effects (font (size 1.27 1.27)) hide)
     )
-    (property "Vendor" "DigiKey" (at 139.065 38.1 0)
-      (effects (font (size 1.27 1.27)) hide)
-    )
-    (property "VendorId" "CT2192LPST-ND" (at 139.065 38.1 0)
+    (property "Vendor" "HTL" (at 139.065 38.1 0)
+      (effects (font (size 1.27 1.27)) hide)
+    )
+    (property "VendorId" "103604" (at 139.065 38.1 0)
       (effects (font (size 1.27 1.27)) hide)
     )
@@
       (effects (font (size 1.27 1.27)) hide)
     )
-    (property "Vendor" "DigiKey" (at 177.8 66.04 0)
-      (effects (font (size 1.27 1.27)) hide)
-    )
-    (property "VendorId" "CKN10891CT-ND" (at 177.8 66.04 0)
-      (effects (font (size 1.27 1.27)) hide)
-    )
+    (property "Vendor" "HTL" (at 177.8 66.04 0)
+      (effects (font (size 1.27 1.27)) hide)
+    )
+    (property "VendorId" "103586" (at 177.8 66.04 0)
+      (effects (font (size 1.27 1.27)) hide)
+    )

Commit message: Adapt values for rng
Parts:
- C12: value 1n -> 1u; VendorId 102542 -> 100134
- C13: value 10n -> 10u; VendorId 102538 -> 100138
- C7, C8, C9: value 100n -> n.B.; Vendor HTL -> (none); VendorId 100128 -> (none)
- R19, R20: value 10k -> 47k; VendorId 102967 -> 102980
Changed lines of the file:
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@@
       (effects (font (size 1.27 1.27)) (justify left))
     )
-    (property "Value" "100n" (at 130.81 179.07 0)
+    (property "Value" "n.B." (at 130.81 179.07 0)
       (effects (font (size 1.27 1.27)) (justify left))
     )
@@
       (effects (font (size 1.27 1.27)) hide)
     )
-    (property "Vendor" "HTL" (at 127 177.8 0)
-      (effects (font (size 1.27 1.27)) hide)
-    )
-    (property "VendorId" "100128" (at 127 177.8 0)
+    (property "Vendor" "" (at 127 177.8 0)
+      (effects (font (size 1.27 1.27)) hide)
+    )
+    (property "VendorId" "" (at 127 177.8 0)
       (effects (font (size 1.27 1.27)) hide)
     )
@@
       (effects (font (size 1.27 1.27)))
     )
-    (property "Value" "10k" (at 226.695 118.11 90)
+    (property "Value" "47k" (at 226.695 118.11 90)
       (effects (font (size 1.27 1.27)))
     )
@@
       (effects (font (size 1.27 1.27)) hide)
     )
-    (property "VendorId" "102967" (at 224.79 123.19 0)
+    (property "VendorId" "102980" (at 224.79 123.19 0)
       (effects (font (size 1.27 1.27)) hide)
     )
@@
       (effects (font (size 1.27 1.27)) (justify left))
     )
-    (property "Value" "10n" (at 228.6 139.7 0)
+    (property "Value" "10u" (at 228.6 139.7 0)
       (effects (font (size 1.27 1.27)) (justify left))
     )
@@
       (effects (font (size 1.27 1.27)) hide)
     )
-    (property "VendorId" "102538" (at 224.79 140.97 0)
+    (property "VendorId" "100138" (at 224.79 140.97 0)
       (effects (font (size 1.27 1.27)) hide)
     )
@@
       (effects (font (size 1.27 1.27)))
     )
-    (property "Value" "10k" (at 221.615 118.11 90)
+    (property "Value" "47k" (at 221.615 118.11 90)
       (effects (font (size 1.27 1.27)))
     )
@@
       (effects (font (size 1.27 1.27)) hide)
     )
-    (property "VendorId" "102967" (at 219.71 123.19 0)
+    (property "VendorId" "102980" (at 219.71 123.19 0)
       (effects (font (size 1.27 1.27)) hide)
     )
@@
       (effects (font (size 1.27 1.27)) (justify left))
     )
-    (property "Value" "1n" (at 215.9 139.7 0)
+    (property "Value" "1u" (at 215.9 139.7 0)
       (effects (font (size 1.27 1.27)) (justify left))
     )
@@
       (effects (font (size 1.27 1.27)) hide)
     )
-    (property "VendorId" "102542" (at 219.71 140.97 0)
+    (property "VendorId" "100134" (at 219.71 140.97 0)
       (effects (font (size 1.27 1.27)) hide)
     )
@@
       (effects (font (size 1.27 1.27)) (justify left))
     )
-    (property "Value" "100n" (at 118.11 179.07 0)
+    (property "Value" "n.B." (at 118.11 179.07 0)
       (effects (font (size 1.27 1.27)) (justify left))
     )
@@
       (effects (font (size 1.27 1.27)) hide)
     )
-    (property "Vendor" "HTL" (at 114.3 177.8 0)
-      (effects (font (size 1.27 1.27)) hide)
-    )
-    (property "VendorId" "100128" (at 114.3 177.8 0)
+    (property "Vendor" "" (at 114.3 177.8 0)
+      (effects (font (size 1.27 1.27)) hide)
+    )
+    (property "VendorId" "" (at 114.3 177.8 0)
       (effects (font (size 1.27 1.27)) hide)
     )
@@
       (effects (font (size 1.27 1.27)) (justify left))
     )
-    (property "Value" "100n" (at 105.41 179.07 0)
+    (property "Value" "n.B." (at 105.41 179.07 0)
       (effects (font (size 1.27 1.27)) (justify left))
     )
@@
       (effects (font (size 1.27 1.27)) hide)
     )
-    (property "Vendor" "HTL" (at 101.6 177.8 0)
-      (effects (font (size 1.27 1.27)) hide)
-    )
-    (property "VendorId" "100128" (at 101.6 177.8 0)
-      (effects (font (size 1.27 1.27)) hide)
-    )
+    (property "Vendor" "" (at 101.6 177.8 0)
+      (effects (font (size 1.27 1.27)) hide)
+    )
+    (property "VendorId" "" (at 101.6 177.8 0)
+      (effects (font (size 1.27 1.27)) hide)
+    )

Commit message: Update to KiCAD 9
Parts:
- FID1, H1, J1, JP1, JP2, TP1: now left out of the parts list
Other:
- moved on the sheet: D2, D3, D4, R14, R15, R5, SW3

Commit message: Rename/Add/Remove bom fields
Parts:
- C1, C2: HTL (none) -> 103620; Vendor HTL -> (none); VendorId 103620 -> (none)
- C10, C3, C4, C5, C6: HTL (none) -> 100128; Vendor HTL -> (none); VendorId 100128 -> (none)
- C11, C13: HTL (none) -> 100138; Vendor HTL -> (none); VendorId 100138 -> (none)
- C12: HTL (none) -> 100134; Vendor HTL -> (none); VendorId 100134 -> (none)
- D1: HTL (none) -> 100194; Vendor HTL -> (none); VendorId 100194 -> (none)
- D2: HTL (none) -> 100206; Vendor HTL -> (none); VendorId 100206 -> (none)
- D3, D5: HTL (none) -> 100458; Vendor HTL -> (none); VendorId 100458 -> (none)
- D4: HTL (none) -> 100459; Vendor HTL -> (none); VendorId 100459 -> (none)
- FB1: HTL (none) -> 103570; Vendor HTL -> (none); VendorId 103570 -> (none)
- H1: HTL (none) -> 101017, 101382; Vendor HTL -> (none); VendorId 101017, 101382 -> (none)
- J1: HTL (none) -> 103572; Vendor HTL -> (none); VendorId 103572 -> (none)
- Q2: HTL (none) -> 103512; Vendor HTL -> (none); VendorId 103512 -> (none)
- R1, R5: HTL (none) -> 102951; Vendor HTL -> (none); VendorId 102951 -> (none)
- R10, R9: HTL (none) -> 102920; Vendor HTL -> (none); VendorId 102920 -> (none)
- R12: HTL (none) -> 102993; Vendor HTL -> (none); VendorId 102993 -> (none)
- R14, R15, R6: HTL (none) -> 102944; Vendor HTL -> (none); VendorId 102944 -> (none)
- R16: HTL (none) -> 102940; Vendor HTL -> (none); VendorId 102940 -> (none)
- R17, R18: HTL (none) -> 102962; Vendor HTL -> (none); VendorId 102962 -> (none)
- R19, R20: HTL (none) -> 102980; Vendor HTL -> (none); VendorId 102980 -> (none)
- R2: HTL (none) -> 102967; Vendor HTL -> (none); VendorId 102967 -> (none)
- R3, R4: HTL (none) -> 102959; Vendor HTL -> (none); VendorId 102959 -> (none)
- R7, R8: HTL (none) -> 102973; Vendor HTL -> (none); VendorId 102973 -> (none)
- SW1, SW2: HTL (none) -> 103586; Vendor HTL -> (none); VendorId 103586 -> (none)
- SW3: HTL (none) -> 103604; Vendor HTL -> (none); VendorId 103604 -> (none)
- U1: HTL (none) -> 103615; Vendor HTL -> (none); VendorId 103615 -> (none)
- U2: HTL (none) -> 103271; Vendor HTL -> (none); VendorId 103271 -> (none)
- U3: HTL (none) -> 103616; Vendor HTL -> (none); VendorId 103616 -> (none)
- U4: HTL (none) -> 103617; Vendor HTL -> (none); VendorId 103617 -> (none)
- U5, U6: HTL (none) -> 103618; Vendor HTL -> (none); VendorId 103618 -> (none)
- U7: HTL (none) -> 103619; Vendor HTL -> (none); VendorId 103619 -> (none)
